Commit message: 11

File: src/fishbot_navigation2/urdf/fishot_2d.urdf (robot description, URDF)
Before this commit: robot cartographer_backpack_3d, 2 links, 1 joints
Links:
- removed link laser
- added link map
- added link odom
- link base_link: geometry visual box size=0.1 0.1 0.1
Joints:
- removed joint laser_joint
- added joint map_to_odom: type fixed, parent map, child odom, origin xyz=0 0 0 rpy=0 0 0
- added joint odom_to_base_link: type fixed, parent odom, child base_link, origin xyz=0 0 0 rpy=0 0 0
